Commit message: robot description

File: tr2_description/urdf/arm/arm.macros.xacro (robot description, xacro)
@@ -2,8 +2,8 @@
 <robot xmlns:xacro="http://www.ros.org/wiki/xacro">
 	<xacro:macro name="arm_link" params="name origin_rpy">
-		<link name="${name}_link">
+		<link name="link_${name}">
 			<collision>
 				<geometry>
-		      <mesh filename="package://tr2_description/meshes/dae/${name}.dae" scale="0.001 0.001 0.001"/>
+		      <mesh filename="package://tr2_description/meshes/stl/link_${name}.stl" scale="0.001 0.001 0.001"/>
 				</geometry>
 				<origin rpy="${origin_rpy}" />
@@ -15,6 +15,9 @@
 			<visual>
 				<geometry>
-		      <mesh filename="package://tr2_description/meshes/dae/${name}.dae" scale="0.001 0.001 0.001"/>
+		      <mesh filename="package://tr2_description/meshes/stl/link_${name}.stl" scale="0.001 0.001 0.001"/>
 				</geometry>
+		    <material name="slate_gray">
+		      <color rgba="0.2 0.2 0.2 1"/>
+		    </material>
 				<origin rpy="${origin_rpy}" />
 			</visual>

File: tr2_description/urdf/arm/arm.urdf.xacro (robot description, xacro)
@@ -4,53 +4,47 @@
   <xacro:include filename="$(find tr2_description)/urdf/arm/arm.gazebo.xacro" />
 	<xacro:include filename="$(find tr2_description)/urdf/arm/arm.transmission.xacro" />
-	<xacro:arm_link name="arm1" origin_rpy="1.5708 0 0" />
-	<xacro:arm_link name="arm2" origin_rpy="1.5708 0 0" />
-	<xacro:arm_link name="arm3" origin_rpy="1.5708 0 0" />
-	<xacro:arm_link name="arm4" origin_rpy="1.5708 0 0" />
-	<xacro:arm_link name="arm5" origin_rpy="-1.5708 3.141592 0" />
-	<xacro:arm_link name="arm6" origin_rpy="-1.5708 0 0" />
-	<joint name="base_to_a0" type="fixed">
+	<xacro:arm_link name="a0" origin_rpy="3.1415 0.0000 1.5708" />
+	<xacro:arm_link name="a1" origin_rpy="1.5708 1.5708 0.0000" />
+	<xacro:arm_link name="a2" origin_rpy="1.5708 0.0000 -1.5708" />
+	<xacro:arm_link name="a3" origin_rpy="1.5708 1.5708 0.0000" />
+	<xacro:arm_link name="g0" origin_rpy="1.5708 0.0000 -1.5708" />
+	<joint name="a0" type="revolute">
 		<parent link="base_link"/>
-		<child link="arm1_link"/>
-		<origin rpy="0 0 1.570796" xyz="0.0 0.15 0.600"/>
-	</joint>
-	<joint name="a0" type="revolute">
-		<parent link="arm1_link"/>
-		<child link="arm2_link"/>
-		<origin xyz="0 0 -0.007"/>
+		<child link="link_a0"/>
+		<origin xyz="0.0933 0.1282 0.7292" rpy="0 3.1415 -1.5708"/>
     <axis xyz="0 0 1"/>
-		<limit effort="1.0" lower="-1" upper="1.5708" velocity="0.2932"/>
+		<limit effort="1.0" lower="-1.8" upper="1.8" velocity="0.2932"/>
     <dynamics damping="0.1" friction="0.1"/>
 	</joint>
 	<joint name="a1" type="revolute">
-		<parent link="arm2_link"/>
-		<child link="arm3_link"/>
-		<origin xyz="0.139238 0 0"/>
+		<parent link="link_a0"/>
+		<child link="link_a1"/>
+		<origin xyz="0.2146 0.0800 -0.0897" rpy="0 3.1415 3.1415"/>
     <axis xyz="0 1 0"/>
-		<limit effort="1.0" lower="-1.5708" upper="1.5708" velocity="0.075"/>
+		<limit effort="1.0" lower="-6.29" upper="6.29" velocity="0.075"/>
     <dynamics damping="0.1" friction="0.1"/>
 	</joint>
 	<joint name="a2" type="revolute">
-		<parent link="arm3_link"/>
-		<child link="arm4_link"/>
-		<origin xyz="0.238827 0 0"/>
+		<parent link="link_a1"/>
+		<child link="link_a2"/>
+		<origin xyz="0.1669 -0.1097 0" rpy="3.1415 3.1415 0"/>
     <axis xyz="1 0 0"/>
-		<limit effort="1.0" lower="-3.1415" upper="3.1415" velocity="0.25"/>
+		<limit effort="1.0" lower="-6.29" upper="6.29" velocity="0.25"/>
     <dynamics damping="0.1" friction="0.1"/>
 	</joint>
 	<joint name="a3" type="revolute">
-		<parent link="arm4_link"/>
-		<child link="arm5_link"/>
-		<origin xyz="0.145 0 0"/>
+		<parent link="link_a2"/>
+		<child link="link_a3"/>
+		<origin xyz="-0.1544 -0.0800 0" rpy="0 3.1415 0"/>
     <axis xyz="0 1 0"/>
-		<limit effort="1.0" lower="-1.75" upper="1.75" velocity="0.1"/>
+		<limit effort="1.0" lower="-6.29" upper="6.29" velocity="0.1"/>
     <dynamics damping="0.1" friction="0.1"/>
 	</joint>
 	<joint name="a4" type="revolute">
-		<parent link="arm5_link"/>
-		<child link="arm6_link"/>
-		<origin xyz="0.230643 0 0"/>
+		<parent link="link_a3"/>
+		<child link="link_g0"/>
+		<origin xyz="0.1669 -0.1097 0" rpy="0 3.1415 0"/>
     <axis xyz="1 0 0"/>
-		<limit effort="1.0" lower="-3.1415" upper="3.1415" velocity="1.4661"/>
+		<limit effort="1.0" lower="-6.29" upper="6.29" velocity="1.4661"/>
     <dynamics damping="0.1" friction="0.1"/>
 	</joint>

File: tr2_description/urdf/base/base.urdf.xacro (robot description, xacro)
@@ -15,7 +15,7 @@
 			<collision>
 				<geometry>
-		      <mesh filename="package://tr2_description/meshes/dae/wheel.dae" scale="0.001 0.001 0.001"/>
+		      <mesh filename="package://tr2_description/meshes/stl/link_b1.stl" scale="0.001 0.001 0.001"/>
 				</geometry>
-				<origin rpy="1.5708 0 0" />
+				<origin rpy="0 0 1.5708" />
 			</collision>
 			<inertial>
@@ -25,7 +25,10 @@
 			<visual>
 				<geometry>
-		      <mesh filename="package://tr2_description/meshes/dae/wheel.dae" scale="0.001 0.001 0.001"/>
+		      <mesh filename="package://tr2_description/meshes/stl/link_b1.stl" scale="0.001 0.001 0.001"/>
 				</geometry>
-				<origin rpy="1.5708 0 0" />
+		    <material name="slate_gray">
+		      <color rgba="0.2 0.2 0.2 1"/>
+		    </material>
+				<origin rpy="0 0 1.5708" />
 			</visual>
 		</link>
@@ -35,7 +38,7 @@
 		<collision>
 			<geometry>
-        <mesh filename="package://tr2_description/meshes/dae/base.dae" scale="0.001 0.001 0.001"/>
+        <mesh filename="package://tr2_description/meshes/stl/link_b0.stl" scale="0.001 0.001 0.001"/>
 			</geometry>
-			<origin rpy="0 0 3.141592" />
+			<origin rpy="0 0 1.5708" />
 		</collision>
 		<inertial>
@@ -45,17 +48,76 @@
 		<visual>
 			<geometry>
-        <mesh filename="package://tr2_description/meshes/dae/base.dae" scale="0.001 0.001 0.001"/>
+        <mesh filename="package://tr2_description/meshes/stl/link_b0.stl" scale="0.001 0.001 0.001"/>
 			</geometry>
-      <material name="white">
-        <color rgba="1 1 1 1"/>
+      <material name="slate_gray">
+        <color rgba="0.2 0.2 0.2 1"/>
       </material>
-			<origin rpy="0 0 3.141592" />
+			<origin rpy="0 0 1.5708" />
 		</visual>
 	</link>
+	<!-- resulting links and joints -->
+	<link name="link_b2">
+		<collision>
+			<geometry>
+        <mesh filename="package://tr2_description/meshes/stl/link_b2.stl" scale="0.001 0.001 0.001"/>
+			</geometry>
+			<origin rpy="0 0 1.5708" />
+		</collision>
+		<inertial>
+			<mass value="1.0"/>
+			<inertia ixx="0.1" iyy="0.1" izz="0.1" ixy="0" ixz="0" iyz="0" />
+		</inertial>
+		<visual>
+			<geometry>
+        <mesh filename="package://tr2_description/meshes/stl/link_b2.stl" scale="0.001 0.001 0.001"/>
+			</geometry>
+      <material name="slate_gray">
+        <color rgba="0.2 0.2 0.2 1"/>
+      </material>
+			<origin rpy="0 0 1.5708" />
+		</visual>
+	</link>
+	<link name="link_b3">
+		<collision>
+			<geometry>
+        <mesh filename="package://tr2_description/meshes/stl/link_b3.stl" scale="0.001 0.001 0.001"/>
+			</geometry>
+			<origin rpy="0 0 1.5708" />
+		</collision>
+		<inertial>
+			<mass value="1.0"/>
+			<inertia ixx="0.1" iyy="0.1" izz="0.1" ixy="0" ixz="0" iyz="0" />
+		</inertial>
+		<visual>
+			<geometry>
+        <mesh filename="package://tr2_description/meshes/stl/link_b3.stl" scale="0.001 0.001 0.001"/>
+			</geometry>
+      <material name="slate_gray">
+        <color rgba="0.2 0.2 0.2 1"/>
+      </material>
+			<origin rpy="0 0 1.5708" />
+		</visual>
+	</link>
+	<joint name="b2" type="continuous">
+		<parent link="base_link"/>
+		<child link="link_b2"/>
+		<origin xyz="0 -0.1960 0" rpy="0 3.1415 -1.5708"/>
+    <axis xyz="0 0 1"/>
+		<limit effort="1.0" lower="-1.8" upper="1.8" velocity="0.2932"/>
+    <dynamics damping="0.1" friction="0.1"/>
+	</joint>
+	<joint name="b3" type="continuous">
+		<parent link="link_b2"/>
+		<child link="link_b3"/>
+		<origin xyz="-0.0138 0 0.0390" rpy="1.5708 0 0"/>
+    <axis xyz="0 0 1"/>
+		<limit effort="1.0" lower="-1.8" upper="1.8" velocity="0.2932"/>
+    <dynamics damping="0.1" friction="0.1"/>
+	</joint>
 	<xacro:tr2_wheel name="b0l">
-		<origin rpy="0 0 -1.570796" xyz="-0.293310 0.0 -0.0725"/>
+		<origin rpy="0 0 -1.570796" xyz="-0.3019 0.1502 0.0508"/>
 	</xacro:tr2_wheel>
 	<xacro:tr2_wheel name="b0r">
-		<origin rpy="0 0 1.570796" xyz="0.293310 0.0 -0.0725"/>
+		<origin rpy="0 0 1.570796" xyz="0.3019 0.1502 0.0508"/>
 	</xacro:tr2_wheel>
 </robot>

File: tr2_description/urdf/head/head.urdf.xacro (robot description, xacro)
@@ -6,7 +6,7 @@
 		<collision>
 			<geometry>
-        <mesh filename="package://tr2_description/meshes/dae/neck.dae" scale="0.001 0.001 0.001"/>
+        <mesh filename="package://tr2_description/meshes/stl/link_h0.stl" scale="0.001 0.001 0.001"/>
 			</geometry>
-			<origin rpy="1.5708 0 0"/>
+			<origin rpy="3.1415 3.1415 0"/>
 		</collision>
 		<inertial>
@@ -16,7 +16,10 @@
 		<visual>
 			<geometry>
-        <mesh filename="package://tr2_description/meshes/dae/neck.dae" scale="0.001 0.001 0.001"/>
+        <mesh filename="package://tr2_description/meshes/stl/link_h0.stl" scale="0.001 0.001 0.001"/>
 			</geometry>
-			<origin rpy="1.5708 0 0"/>
+	    <material name="slate_gray">
+	      <color rgba="0.2 0.2 0.2 1"/>
+	    </material>
+			<origin rpy="3.1415 3.1415 0"/>
 		</visual>
 	</link>
@@ -24,7 +27,7 @@
 		<collision>
 			<geometry>
-        <mesh filename="package://tr2_description/meshes/dae/head.dae" scale="0.001 0.001 0.001"/>
+        <mesh filename="package://tr2_description/meshes/stl/link_h1.stl" scale="0.001 0.001 0.001"/>
 			</geometry>
-			<origin rpy="1.5708 0 0"/>
+			<origin rpy="0 3.1415 0"/>
 		</collision>
 		<inertial>
@@ -34,7 +37,10 @@
 		<visual>
 			<geometry>
-        <mesh filename="package://tr2_description/meshes/dae/head.dae" scale="0.001 0.001 0.001"/>
+        <mesh filename="package://tr2_description/meshes/stl/link_h1.stl" scale="0.001 0.001 0.001"/>
 			</geometry>
-			<origin rpy="0 -1.5708 -1.5708"/>
+	    <material name="slate_gray">
+	      <color rgba="0.2 0.2 0.2 1"/>
+	    </material>
+			<origin rpy="0 3.1415 0"/>
 		</visual>
 	</link>
@@ -60,5 +66,5 @@
 		<parent link="base_link"/>
 		<child link="neck_link"/>
-		<origin xyz="0 -0.017 0.850"/>
+		<origin xyz="0 -0.1227 0.9071"/>
     <axis xyz="0 0 1"/>
 		<limit effort="1.0" lower="-1.5708" upper="1.5708" velocity="0.5"/>
@@ -68,5 +74,5 @@
 		<parent link="neck_link"/>
 		<child link="head_link"/>
-		<origin xyz="0 0.090789 0.09"/>
+		<origin xyz="-0.0688 0.1745 0.1614" rpy="-0.3490 0 0"/>
     <axis xyz="1 0 0"/>
 		<limit effort="1.0" lower="-0.75" upper="0.4" velocity="0.5"/>
