Commit message: base wheel integration, gripper integration

File: tr2_description/urdf/arm/arm.gazebo.xacro (robot description, xacro)
@@ -2,4 +2,5 @@
 <robot xmlns:xacro="http://www.ros.org/wiki/xacro">
   <xacro:include filename="$(find tr2_description)/urdf/arm/arm.macros.xacro" />
+	<xacro:mimic_joint parent="g0" joint="g0_b" multiplier="-1"/>
 	<gazebo reference="link_a0">
 		<material>Gazebo/DarkGrey</material>

File: tr2_description/urdf/arm/arm.transmission.xacro (robot description, xacro)
@@ -7,3 +7,4 @@
 	<xacro:arm_trans joint_name="a3" />
 	<xacro:arm_trans joint_name="a4" />
+	<xacro:arm_trans joint_name="g0" />
 </robot>

File: tr2_description/urdf/arm/arm.urdf.xacro (robot description, xacro)
@@ -56,5 +56,5 @@
 		<origin rpy="0 0 0" xyz="-0.135 0.0075 0"/>
     <axis xyz="0 1 0"/>
-		<limit effort="1.0" lower="0" upper="0.041" velocity="0.5"/>
+		<limit effort="1.0" lower="0" upper="0.041" velocity="0.01"/>
     <dynamics damping="0.1" friction="0.1"/>
 	</joint>
@@ -64,5 +64,6 @@
 		<origin rpy="0 0 0" xyz="-0.135 -0.0075 0"/>
     <axis xyz="0 1 0"/>
-		<limit effort="1.0" lower="-0.041" upper="0" velocity="0.5"/>
+		<mimic joint="g0" multiplier="-1" offset="0"/>
+		<limit effort="1.0" lower="-0.041" upper="0" velocity="0.01"/>
     <dynamics damping="0.1" friction="0.1"/>
 	</joint>

File: tr2_description/urdf/base/base.gazebo.xacro (robot description, xacro)
@@ -3,4 +3,22 @@
 	<gazebo reference="link_b0">
 		<material>Gazebo/DarkGrey</material>
+		<collision>
+      <surface>
+			  <contact>
+		      <ode>
+		        <kp>1e15</kp>
+		        <kd>1e13</kd>
+		      </ode>
+		    </contact>
+        <friction>
+          <ode>
+            <mu>100000.0</mu>
+            <mu2>100000.0</mu2>
+            <slip1>0.0</slip1>
+            <slip2>0.0</slip2>
+          </ode>
+        </friction>
+      </surface>
+		</collision>
 	</gazebo>
 	<gazebo reference="base_link">
@@ -9,4 +27,22 @@
 	<gazebo reference="link_b1">
 		<material>Gazebo/DarkGrey</material>
+		<collision>
+      <surface>
+			  <contact>
+		      <ode>
+		        <kp>1e15</kp>
+		        <kd>1e13</kd>
+		      </ode>
+		    </contact>
+        <friction>
+          <ode>
+            <mu>100000.0</mu>
+            <mu2>100000.0</mu2>
+            <slip1>0.0</slip1>
+            <slip2>0.0</slip2>
+          </ode>
+        </friction>
+      </surface>
+		</collision>
 	</gazebo>
 	<gazebo reference="link_b2">

File: tr2_description/urdf/base/base.urdf.xacro (robot description, xacro)
@@ -9,7 +9,7 @@
 			<child link="link_${name}"/>
 		  <axis xyz="0 1 0"/>
-			<limit effort="1.0" lower="-1.0" upper="1.0" velocity="12.0"/>
+			<limit effort="100.0" lower="-12.0" upper="12.0" velocity="12.0"/>
 			<xacro:insert_block name="origin" />
-    	<dynamics damping="0" friction="0"/>
+    	<dynamics damping="1.0" friction="1.0"/>
 		</joint>
 		<link name="link_${name}">
@@ -21,5 +21,5 @@
 			</collision>
 			<inertial>
-				<mass value="1.0"/>
+				<mass value="12.0"/>
 				<inertia ixx="0.1" iyy="0.1" izz="0.1" ixy="0" ixz="0" iyz="0" />
 			</inertial>
