Commit message: moveit integration, tr2py development

File: tr2_description/urdf/arm/arm.urdf.xacro (robot description, xacro)
@@ -9,4 +9,6 @@
 	<xacro:arm_link name="a3" origin_rpy="1.5708 1.5708 0.0000" />
 	<xacro:arm_link name="g0" origin_rpy="1.5708 0.0000 -1.5708" />
+	<xacro:arm_link name="g1" origin_rpy="1.5708 -1.5708 0.0000" />
+	<xacro:arm_link name="g1_b" origin_rpy="1.5708 -1.5708 0.0000" />
 	<joint name="a0" type="revolute">
 		<parent link="base_link"/>
@@ -14,5 +16,5 @@
 		<origin xyz="0.0933 0.1282 0.7292" rpy="0 3.1415 -1.5708"/>
     <axis xyz="0 0 1"/>
-		<limit effort="1.0" lower="-1.8" upper="1.8" velocity="0.2932"/>
+		<limit effort="1.0" lower="-15" upper="15" velocity="0.42"/>
     <dynamics damping="0.1" friction="0.1"/>
 	</joint>
@@ -22,5 +24,5 @@
 		<origin xyz="0.2146 0.0800 -0.0897" rpy="0 3.1415 3.1415"/>
     <axis xyz="0 1 0"/>
-		<limit effort="1.0" lower="-6.29" upper="6.29" velocity="0.075"/>
+		<limit effort="1.0" lower="-15" upper="15" velocity="0.42"/>
     <dynamics damping="0.1" friction="0.1"/>
 	</joint>
@@ -30,5 +32,5 @@
 		<origin xyz="0.1669 -0.1097 0" rpy="3.1415 3.1415 0"/>
     <axis xyz="1 0 0"/>
-		<limit effort="1.0" lower="-6.29" upper="6.29" velocity="0.25"/>
+		<limit effort="1.0" lower="-15" upper="15" velocity="0.42"/>
     <dynamics damping="0.1" friction="0.1"/>
 	</joint>
@@ -38,5 +40,5 @@
 		<origin xyz="-0.1544 -0.0800 0" rpy="0 3.1415 0"/>
     <axis xyz="0 1 0"/>
-		<limit effort="1.0" lower="-6.29" upper="6.29" velocity="0.1"/>
+		<limit effort="1.0" lower="-15" upper="15" velocity="0.42"/>
     <dynamics damping="0.1" friction="0.1"/>
 	</joint>
@@ -46,14 +48,22 @@
 		<origin xyz="0.1669 -0.1097 0" rpy="0 3.1415 0"/>
     <axis xyz="1 0 0"/>
-		<limit effort="1.0" lower="-6.29" upper="6.29" velocity="1.4661"/>
+		<limit effort="1.0" lower="-15" upper="15" velocity="0.42"/>
     <dynamics damping="0.1" friction="0.1"/>
 	</joint>
-	<!--<joint name="g0" type="revolute">
-		<parent link="gripper1_link"/>
-		<child link="gripper2_link"/>
-		<origin rpy="0 0 -1.5708" xyz="0.024 -0.014 0"/>
-    <axis xyz="0 0 1"/>
-		<limit effort="1.0" lower="0" upper="1.5708" velocity="0.5"/>
+	<joint name="g0" type="prismatic">
+		<parent link="link_g0"/>
+		<child link="link_g1"/>
+		<origin rpy="0 0 0" xyz="-0.135 0.0075 0"/>
+    <axis xyz="0 1 0"/>
+		<limit effort="1.0" lower="0" upper="0.041" velocity="0.5"/>
     <dynamics damping="0.1" friction="0.1"/>
-	</joint>-->
+	</joint>
+	<joint name="g0_b" type="prismatic">
+		<parent link="link_g0"/>
+		<child link="link_g1_b"/>
+		<origin rpy="0 0 0" xyz="-0.135 -0.0075 0"/>
+    <axis xyz="0 1 0"/>
+		<limit effort="1.0" lower="-0.041" upper="0" velocity="0.5"/>
+    <dynamics damping="0.1" friction="0.1"/>
+	</joint>
 </robot>

File: tr2_description/urdf/head/head.urdf.xacro (robot description, xacro)
@@ -68,5 +68,5 @@
 		<origin xyz="0 -0.1227 0.9071"/>
     <axis xyz="0 0 1"/>
-		<limit effort="1.0" lower="-1.5708" upper="1.5708" velocity="0.5"/>
+		<limit effort="1.0" lower="-6.29" upper="6.29" velocity="1.4661"/>
     <dynamics damping="0.1" friction="0.1"/>
 	</joint>
@@ -76,5 +76,5 @@
 		<origin xyz="-0.0688 0.1745 0.1614" rpy="-0.3490 0 0"/>
     <axis xyz="1 0 0"/>
-		<limit effort="1.0" lower="-0.75" upper="0.4" velocity="0.5"/>
+		<limit effort="1.0" lower="-6.29" upper="6.29" velocity="1.4661"/>
     <dynamics damping="0.1" friction="0.1"/>
 	</joint>

Commit message: gazebo integration

File: tr2_description/urdf/arm/arm.urdf.xacro (robot description, xacro)
@@ -16,5 +16,5 @@
 		<origin xyz="0.0933 0.1282 0.7292" rpy="0 3.1415 -1.5708"/>
     <axis xyz="0 0 1"/>
-		<limit effort="1.0" lower="-15" upper="15" velocity="0.42"/>
+		<limit effort="1.0" lower="-15" upper="15" velocity="0.30"/>
     <dynamics damping="0.1" friction="0.1"/>
 	</joint>
@@ -24,5 +24,5 @@
 		<origin xyz="0.2146 0.0800 -0.0897" rpy="0 3.1415 3.1415"/>
     <axis xyz="0 1 0"/>
-		<limit effort="1.0" lower="-15" upper="15" velocity="0.42"/>
+		<limit effort="1.0" lower="-15" upper="15" velocity="0.30"/>
     <dynamics damping="0.1" friction="0.1"/>
 	</joint>
@@ -32,5 +32,5 @@
 		<origin xyz="0.1669 -0.1097 0" rpy="3.1415 3.1415 0"/>
     <axis xyz="1 0 0"/>
-		<limit effort="1.0" lower="-15" upper="15" velocity="0.42"/>
+		<limit effort="1.0" lower="-15" upper="15" velocity="0.30"/>
     <dynamics damping="0.1" friction="0.1"/>
 	</joint>
@@ -40,5 +40,5 @@
 		<origin xyz="-0.1544 -0.0800 0" rpy="0 3.1415 0"/>
     <axis xyz="0 1 0"/>
-		<limit effort="1.0" lower="-15" upper="15" velocity="0.42"/>
+		<limit effort="1.0" lower="-15" upper="15" velocity="0.30"/>
     <dynamics damping="0.1" friction="0.1"/>
 	</joint>
@@ -48,5 +48,5 @@
 		<origin xyz="0.1669 -0.1097 0" rpy="0 3.1415 0"/>
     <axis xyz="1 0 0"/>
-		<limit effort="1.0" lower="-15" upper="15" velocity="0.42"/>
+		<limit effort="1.0" lower="-15" upper="15" velocity="0.30"/>
     <dynamics damping="0.1" friction="0.1"/>
 	</joint>

Commit message: joint behavior, limits

File: tr2_description/urdf/arm/arm.urdf.xacro (robot description, xacro)
@@ -16,5 +16,5 @@
 		<origin xyz="0.0933 0.1282 0.7292" rpy="0 3.1415 -1.5708"/>
     <axis xyz="0 0 1"/>
-		<limit effort="1.0" lower="-15" upper="15" velocity="0.30"/>
+		<limit effort="100.0" lower="-2" upper="2" velocity="0.20"/>
     <dynamics damping="0.1" friction="0.1"/>
 	</joint>
@@ -24,5 +24,5 @@
 		<origin xyz="0.2146 0.0800 -0.0897" rpy="0 3.1415 3.1415"/>
     <axis xyz="0 1 0"/>
-		<limit effort="1.0" lower="-15" upper="15" velocity="0.30"/>
+		<limit effort="100.0" lower="-15" upper="15" velocity="0.20"/>
     <dynamics damping="0.1" friction="0.1"/>
 	</joint>
@@ -32,5 +32,5 @@
 		<origin xyz="0.1669 -0.1097 0" rpy="3.1415 3.1415 0"/>
     <axis xyz="1 0 0"/>
-		<limit effort="1.0" lower="-15" upper="15" velocity="0.30"/>
+		<limit effort="100.0" lower="-15" upper="15" velocity="0.20"/>
     <dynamics damping="0.1" friction="0.1"/>
 	</joint>
@@ -40,5 +40,5 @@
 		<origin xyz="-0.1544 -0.0800 0" rpy="0 3.1415 0"/>
     <axis xyz="0 1 0"/>
-		<limit effort="1.0" lower="-15" upper="15" velocity="0.30"/>
+		<limit effort="100.0" lower="-15" upper="15" velocity="0.20"/>
     <dynamics damping="0.1" friction="0.1"/>
 	</joint>
@@ -48,5 +48,5 @@
 		<origin xyz="0.1669 -0.1097 0" rpy="0 3.1415 0"/>
     <axis xyz="1 0 0"/>
-		<limit effort="1.0" lower="-15" upper="15" velocity="0.30"/>
+		<limit effort="100.0" lower="-15" upper="15" velocity="0.20"/>
     <dynamics damping="0.1" friction="0.1"/>
 	</joint>
@@ -56,5 +56,5 @@
 		<origin rpy="0 0 0" xyz="-0.135 0.0075 0"/>
     <axis xyz="0 1 0"/>
-		<limit effort="1.0" lower="0" upper="0.041" velocity="0.01"/>
+		<limit effort="100.0" lower="0" upper="0.041" velocity="0.01"/>
     <dynamics damping="0.1" friction="0.1"/>
 	</joint>
@@ -65,5 +65,5 @@
     <axis xyz="0 1 0"/>
 		<mimic joint="g0" multiplier="-1" offset="0"/>
-		<limit effort="1.0" lower="-0.041" upper="0" velocity="0.01"/>
+		<limit effort="100.0" lower="-0.041" upper="0" velocity="0.01"/>
     <dynamics damping="0.1" friction="0.1"/>
 	</joint>

File: tr2_description/urdf/base/base.urdf.xacro (robot description, xacro)
@@ -9,7 +9,7 @@
 			<child link="link_${name}"/>
 		  <axis xyz="0 1 0"/>
-			<limit effort="100.0" lower="-12.0" upper="12.0" velocity="12.0"/>
+			<limit effort="100.0" lower="-4.0" upper="4.0" velocity="4.0"/>
 			<xacro:insert_block name="origin" />
-    	<dynamics damping="1.0" friction="1.0"/>
+    	<dynamics damping="1.0" friction="2.0"/>
 		</joint>
 		<link name="link_${name}">

Commit message: created tr2_node class, joint_sim class

File: tr2_description/urdf/arm/arm.urdf.xacro (robot description, xacro)
@@ -14,5 +14,5 @@
 		<parent link="base_link"/>
 		<child link="link_a0"/>
-		<origin xyz="0.0933 0.1282 0.7292" rpy="0 3.1415 -1.5708"/>
+		<origin xyz="0.0933 0.1282 0.7292" rpy="0 3.1415 0"/>
     <axis xyz="0 0 1"/>
 		<limit effort="100.0" lower="-2" upper="2" velocity="0.20"/>
@@ -22,5 +22,5 @@
 		<parent link="link_a0"/>
 		<child link="link_a1"/>
-		<origin xyz="0.2146 0.0800 -0.0897" rpy="0 3.1415 3.1415"/>
+		<origin xyz="0.2146 0.0800 -0.0897" rpy="0 -1.5708 3.1415"/>
     <axis xyz="0 1 0"/>
 		<limit effort="100.0" lower="-15" upper="15" velocity="0.20"/>
@@ -38,5 +38,5 @@
 		<parent link="link_a2"/>
 		<child link="link_a3"/>
-		<origin xyz="-0.1544 -0.0800 0" rpy="0 3.1415 0"/>
+		<origin xyz="-0.1544 -0.0800 0" rpy="0 1.5708 0"/>
     <axis xyz="0 1 0"/>
 		<limit effort="100.0" lower="-15" upper="15" velocity="0.20"/>
@@ -46,5 +46,5 @@
 		<parent link="link_a3"/>
 		<child link="link_g0"/>
-		<origin xyz="0.1669 -0.1097 0" rpy="0 3.1415 0"/>
+		<origin xyz="0.1669 -0.1097 0" rpy="0.5236 3.1415 0"/>
     <axis xyz="1 0 0"/>
 		<limit effort="100.0" lower="-15" upper="15" velocity="0.20"/>
