Commit message: tr2 xacro file, wip

File: tr2_description/robots/tr2.urdf.xacro (robot description, xacro)
@@ -3,8 +3,7 @@
 	<xacro:property name="M_PI" value="3.141509" />
 	<xacro:include filename="$(find tr2_description)/urdf/base/base.urdf.xacro"/>
-	<xacro:include filename="$(find tr2_description)/urdf/body/body.urdf.xacro"/>
+	<!--<xacro:include filename="$(find tr2_description)/urdf/body/body.urdf.xacro"/>-->
 	<xacro:include filename="$(find tr2_description)/urdf/head/head.urdf.xacro"/>
-	<xacro:include filename="$(find tr2_description)/urdf/arm/right_arm.urdf.xacro"/>
-	<xacro:include filename="$(find tr2_description)/urdf/arm/left_arm.urdf.xacro"/>
+	<xacro:include filename="$(find tr2_description)/urdf/arm/arm.urdf.xacro"/>
   <gazebo>
     <plugin name="gazebo_ros_control" filename="libgazebo_ros_control.so">

File: tr2_description/urdf/arm/arm.macros.xacro (robot description, xacro)
@@ -1,6 +1,6 @@
 <?xml version="1.0"?>
 <robot xmlns:xacro="http://www.ros.org/wiki/xacro">
-	<xacro:macro name="arm_link" params="prefix name origin_rpy">
-		<link name="${prefix}_${name}_link">
+	<xacro:macro name="arm_link" params="name origin_rpy">
+		<link name="${name}_link">
 			<collision>
 				<geometry>

File: tr2_description/urdf/base/base.transmission.xacro (robot description, xacro)
@@ -1,5 +1,5 @@
 <?xml version="1.0"?>
 <robot xmlns:xacro="http://www.ros.org/wiki/xacro">
-  <transmission name="JointBaseWheelFR_trans">
+  <transmission name="b0l_trans">
     <type>transmission_interface/SimpleTransmission</type>
     <actuator name="motor19">
@@ -7,9 +7,9 @@
       <hardwareInterface>EffortJointInterface</hardwareInterface>
     </actuator>
-    <joint name="JointBaseWheelFR">
+    <joint name="b0l">
       <hardwareInterface>hardware_interface/EffortJointInterface</hardwareInterface>
     </joint>
   </transmission>
-  <transmission name="JointBaseWheelFL_trans">
+  <transmission name="b0r_trans">
     <type>transmission_interface/SimpleTransmission</type>
     <actuator name="motor20">
@@ -17,35 +17,5 @@
       <hardwareInterface>EffortJointInterface</hardwareInterface>
     </actuator>
-    <joint name="JointBaseWheelFL">
-      <hardwareInterface>hardware_interface/EffortJointInterface</hardwareInterface>
-    </joint>
-  </transmission>
-  <transmission name="JointBaseWheelBR_trans">
-    <type>transmission_interface/SimpleTransmission</type>
-    <actuator name="motor21">
-      <mechanicalReduction>1</mechanicalReduction>
-      <hardwareInterface>EffortJointInterface</hardwareInterface>
-    </actuator>
-    <joint name="JointBaseWheelBR">
-      <hardwareInterface>hardware_interface/EffortJointInterface</hardwareInterface>
-    </joint>
-  </transmission>
-  <transmission name="JointBaseWheelBL_trans">
-    <type>transmission_interface/SimpleTransmission</type>
-    <actuator name="motor22">
-      <mechanicalReduction>1</mechanicalReduction>
-      <hardwareInterface>EffortJointInterface</hardwareInterface>
-    </actuator>
-    <joint name="JointBaseWheelBL">
-      <hardwareInterface>hardware_interface/EffortJointInterface</hardwareInterface>
-    </joint>
-  </transmission>
-  <transmission name="JointTorsoExtension_trans">
-    <type>transmission_interface/SimpleTransmission</type>
-    <actuator name="motor23">
-      <mechanicalReduction>1</mechanicalReduction>
-      <hardwareInterface>EffortJointInterface</hardwareInterface>
-    </actuator>
-    <joint name="JointTorsoExtension">
+    <joint name="b0r">
       <hardwareInterface>hardware_interface/EffortJointInterface</hardwareInterface>
     </joint>

File: tr2_description/urdf/base/base.urdf.xacro (robot description, xacro)
@@ -3,42 +3,7 @@
   <xacro:include filename="$(find tr2_description)/urdf/base/base.gazebo.xacro" />
 	<xacro:include filename="$(find tr2_description)/urdf/base/base.transmission.xacro" />
-	<!-- roller macros -->
-	<xacro:macro name="wheel_rollers" params="i total parent radius">
-		<xacro:property name="wheel_roller_angle" value="${i / total * pi * 2}" />
-		<xacro:property name="wheel_roller_rpy" value="0 ${(pi / 2) + wheel_roller_angle} 0" />
-		<xacro:property name="wheel_roller_xyz" value="${radius * sin(wheel_roller_angle)} 0 ${radius * cos(wheel_roller_angle)}" />
-		<joint name="${parent}_roller_${i + 1}_joint" type="continuous">
-			<parent link="${parent}_link"/>
-			<child link="${parent}_roller_${i + 1}_link"/>
-		  <axis xyz="0 0 1"/>
-			<origin rpy="${wheel_roller_rpy}" xyz="${wheel_roller_xyz}"/>
-			<xacro:insert_block name="origin" />
-    	<dynamics damping="0.1" friction="0.1"/>
-		</joint>
-		<link name="${parent}_roller_${i + 1}_link">
-			<collision>
-				<geometry>
-		      <cylinder length="0.02" radius="0.005" />
-				</geometry>
-				<origin rpy="0 0 0" xyz="0 0 0"/>
-			</collision>
-			<inertial>
-				<mass value="0.001"/>
-				<inertia ixx="0.001" iyy="0.001" izz="0.001" ixy="0" ixz="0" iyz="0" />
-			</inertial>
-			<visual>
-				<geometry>
-		      <cylinder length="0.02" radius="0.005" />
-				</geometry>
-				<origin rpy="0 0 0" xyz="0 0 0"/>
-			</visual>
-		</link>
-		<xacro:if value="${total - i - 1}">
-			<xacro:wheel_rollers i="${i + 1}" total="${total}" parent="${parent}" radius="${radius}" />
-		</xacro:if>
-	</xacro:macro>
 	<!-- wheel macros -->
   <xacro:macro name="tr2_wheel" params="name *origin">
-		<joint name="Joint${name}" type="continuous">
+		<joint name="${name}" type="continuous">
 			<parent link="base_link"/>
 			<child link="${name}_link"/>
@@ -48,10 +13,10 @@
 		</joint>
 		<link name="${name}_link">
-			<!--<collision>
+			<collision>
 				<geometry>
 		      <mesh filename="package://tr2_description/meshes/dae/wheel.dae" scale="0.001 0.001 0.001"/>
 				</geometry>
 				<origin rpy="1.5708 0 0" />
-			</collision>-->
+			</collision>
 			<inertial>
 				<mass value="1.0"/>
@@ -65,5 +30,4 @@
 			</visual>
 		</link>
-		<xacro:wheel_rollers i="0" total="12" parent="${name}" radius="0.068" />
 	</xacro:macro>
 	<!-- resulting links and joints -->
@@ -89,23 +53,9 @@
 		</visual>
 	</link>
-	<joint name="JointTorsoExtension" type="prismatic">
-		<parent link="base_link"/>
-		<child link="body_link"/>
-    <axis xyz="0 0 1"/>
-		<limit effort="1000.0" lower="0" upper="0.150" velocity="0.0001"/>
-		<origin xyz="0 0 0.707"/>
-    <dynamics damping="0.1" friction="0.1"/>
-	</joint>
-	<xacro:tr2_wheel name="BaseWheelFL">
-		<origin rpy="0 0 0.785398" xyz="-0.293310 0.417810 -0.0725"/>
+	<xacro:tr2_wheel name="b0l">
+		<origin rpy="0 0 -1.570796" xyz="-0.293310 0.0 -0.0725"/>
 	</xacro:tr2_wheel>
-	<xacro:tr2_wheel name="BaseWheelFR">
-		<origin rpy="0 0 -0.785398" xyz="0.293310 0.417810 -0.0725"/>
-	</xacro:tr2_wheel>
-	<xacro:tr2_wheel name="BaseWheelBL">
-		<origin rpy="0 0 0.785398" xyz="0.293310 -0.168810 -0.0725"/>
-	</xacro:tr2_wheel>
-	<xacro:tr2_wheel name="BaseWheelBR">
-		<origin rpy="0 0 -0.785398" xyz="-0.293310 -0.168810 -0.0725"/>
+	<xacro:tr2_wheel name="b0r">
+		<origin rpy="0 0 1.570796" xyz="0.293310 0.0 -0.0725"/>
 	</xacro:tr2_wheel>
 </robot>

File: tr2_description/urdf/head/head.transmission.xacro (robot description, xacro)
@@ -1,21 +1,21 @@
 <?xml version="1.0"?>
 <robot xmlns:xacro="http://www.ros.org/wiki/xacro">
-  <transmission name="HeadTilt_trans">
+  <transmission name="h0_trans">
     <type>transmission_interface/SimpleTransmission</type>
-    <actuator name="JointHeadTilt_actuator">
+    <actuator name="h0_actuator">
       <mechanicalReduction>378</mechanicalReduction>
       <hardwareInterface>EffortJointInterface</hardwareInterface>
     </actuator>
-    <joint name="JointHeadTilt">
+    <joint name="h0">
       <hardwareInterface>hardware_interface/EffortJointInterface</hardwareInterface>
     </joint>
   </transmission>
-  <transmission name="HeadPan_trans">
+  <transmission name="h1_trans">
     <type>transmission_interface/SimpleTransmission</type>
-    <actuator name="JointHeadPan_actuator">
+    <actuator name="h1_actuator">
       <mechanicalReduction>378</mechanicalReduction>
       <hardwareInterface>EffortJointInterface</hardwareInterface>
     </actuator>
-    <joint name="JointHeadPan">
+    <joint name="h1">
       <hardwareInterface>hardware_interface/EffortJointInterface</hardwareInterface>
     </joint>

File: tr2_description/urdf/head/head.urdf.xacro (robot description, xacro)
@@ -3,22 +3,4 @@
   <xacro:include filename="$(find tr2_description)/urdf/head/head.gazebo.xacro" />
 	<xacro:include filename="$(find tr2_description)/urdf/head/head.transmission.xacro" />
-	<link name="neck_base_link">
-		<collision>
-			<geometry>
-        <mesh filename="package://tr2_description/meshes/dae/neck_base.dae" scale="0.001 0.001 0.001"/>
-			</geometry>
-			<origin rpy="1.5708 0 0"/>
-		</collision>
-		<inertial>
-			<mass value="0.005"/>
-			<inertia ixx="0.001" iyy="0.001" izz="0.001" ixy="0" ixz="0" iyz="0" />
-		</inertial>
-		<visual>
-			<geometry>
-        <mesh filename="package://tr2_description/meshes/dae/neck_base.dae" scale="0.001 0.001 0.001"/>
-			</geometry>
-			<origin rpy="1.5708 0 0"/>
-		</visual>
-	</link>
 	<link name="neck_link">
 		<collision>
@@ -75,13 +57,13 @@
 		<axis xyz="1 0 0" />
 	</joint>
-	<joint name="JointHeadPan" type="revolute">
-		<parent link="neck_base_link"/>
+	<joint name="h0" type="revolute">
+		<parent link="base_link"/>
 		<child link="neck_link"/>
-		<origin xyz="0 0 0.035"/>
+		<origin xyz="0 -0.017 0.850"/>
     <axis xyz="0 0 1"/>
 		<limit effort="1.0" lower="-1.5708" upper="1.5708" velocity="0.5"/>
     <dynamics damping="0.1" friction="0.1"/>
 	</joint>
-	<joint name="JointHeadTilt" type="revolute">
+	<joint name="h1" type="revolute">
 		<parent link="neck_link"/>
 		<child link="head_link"/>

Commit message: gazebo integration

File: tr2_description/robots/tr2.urdf.xacro (robot description, xacro)
@@ -6,8 +6,10 @@
 	<xacro:include filename="$(find tr2_description)/urdf/head/head.urdf.xacro"/>
 	<xacro:include filename="$(find tr2_description)/urdf/arm/arm.urdf.xacro"/>
-  <gazebo>
-    <plugin name="gazebo_ros_control" filename="libgazebo_ros_control.so">
-      <robotNamespace>/</robotNamespace>
-    </plugin>
+	<gazebo>
+		<plugin name="gazebo_ros_control" filename="libgazebo_ros_control.so">
+			<robotNamespace>/</robotNamespace>
+			<robotSimType>gazebo_ros_control/DefaultRobotHWSim</robotSimType>
+			<legacyModeNS>true</legacyModeNS>
+		</plugin>
 	</gazebo>
 </robot>

File: tr2_description/urdf/base/base.transmission.xacro (robot description, xacro)
@@ -1,5 +1,5 @@
 <?xml version="1.0"?>
 <robot xmlns:xacro="http://www.ros.org/wiki/xacro">
-  <transmission name="b0l_trans">
+  <transmission name="b0_trans">
     <type>transmission_interface/SimpleTransmission</type>
     <actuator name="motor19">
@@ -7,9 +7,9 @@
       <hardwareInterface>EffortJointInterface</hardwareInterface>
     </actuator>
-    <joint name="b0l">
+    <joint name="b0">
       <hardwareInterface>hardware_interface/EffortJointInterface</hardwareInterface>
     </joint>
   </transmission>
-  <transmission name="b0r_trans">
+  <transmission name="b1_trans">
     <type>transmission_interface/SimpleTransmission</type>
     <actuator name="motor20">
@@ -17,5 +17,5 @@
       <hardwareInterface>EffortJointInterface</hardwareInterface>
     </actuator>
-    <joint name="b0r">
+    <joint name="b1">
       <hardwareInterface>hardware_interface/EffortJointInterface</hardwareInterface>
     </joint>

File: tr2_description/urdf/base/base.urdf.xacro (robot description, xacro)
@@ -9,6 +9,7 @@
 			<child link="${name}_link"/>
 		  <axis xyz="0 1 0"/>
+			<limit effort="1.0" lower="-1.0" upper="1.0" velocity="12.0"/>
 			<xacro:insert_block name="origin" />
-    	<dynamics damping="0.1" friction="0.1"/>
+    	<dynamics damping="0" friction="0"/>
 		</joint>
 		<link name="${name}_link">
@@ -104,5 +105,4 @@
 		<origin xyz="0 -0.1960 0" rpy="0 3.1415 -1.5708"/>
     <axis xyz="0 0 1"/>
-		<limit effort="1.0" lower="-1.8" upper="1.8" velocity="0.2932"/>
     <dynamics damping="0.1" friction="0.1"/>
 	</joint>
@@ -112,11 +112,10 @@
 		<origin xyz="-0.0138 0 0.0390" rpy="1.5708 0 0"/>
     <axis xyz="0 0 1"/>
-		<limit effort="1.0" lower="-1.8" upper="1.8" velocity="0.2932"/>
     <dynamics damping="0.1" friction="0.1"/>
 	</joint>
-	<xacro:tr2_wheel name="b0l">
-		<origin rpy="0 0 -1.570796" xyz="-0.3019 0.1502 0.0508"/>
+	<xacro:tr2_wheel name="b0">
+		<origin rpy="0 0 1.570796" xyz="-0.3019 0.1502 0.0508"/>
 	</xacro:tr2_wheel>
-	<xacro:tr2_wheel name="b0r">
+	<xacro:tr2_wheel name="b1">
 		<origin rpy="0 0 1.570796" xyz="0.3019 0.1502 0.0508"/>
 	</xacro:tr2_wheel>

Commit message: gazebo colors, integration

File: tr2_description/robots/tr2.urdf.xacro (robot description, xacro)
@@ -12,4 +12,5 @@
 			<legacyModeNS>true</legacyModeNS>
 		</plugin>
+    <material>Gazebo/LightGrey</material>
 	</gazebo>
 </robot>

File: tr2_description/urdf/arm/arm.gazebo.xacro (robot description, xacro)
@@ -2,3 +2,24 @@
 <robot xmlns:xacro="http://www.ros.org/wiki/xacro">
   <xacro:include filename="$(find tr2_description)/urdf/arm/arm.macros.xacro" />
+	<gazebo reference="link_a0">
+		<material>Gazebo/DarkGrey</material>
+	</gazebo>
+	<gazebo reference="link_a1">
+		<material>Gazebo/DarkGrey</material>
+	</gazebo>
+	<gazebo reference="link_a2">
+		<material>Gazebo/DarkGrey</material>
+	</gazebo>
+	<gazebo reference="link_a3">
+		<material>Gazebo/DarkGrey</material>
+	</gazebo>
+	<gazebo reference="link_g0">
+		<material>Gazebo/DarkGrey</material>
+	</gazebo>
+	<gazebo reference="link_g1">
+		<material>Gazebo/DarkGrey</material>
+	</gazebo>
+	<gazebo reference="link_g1_b">
+		<material>Gazebo/DarkGrey</material>
+	</gazebo>
 </robot>

File: tr2_description/urdf/base/base.gazebo.xacro (robot description, xacro)
@@ -1,3 +1,18 @@
 <?xml version="1.0"?>
 <robot xmlns:xacro="http://www.ros.org/wiki/xacro">
+	<gazebo reference="link_b0">
+		<material>Gazebo/DarkGrey</material>
+	</gazebo>
+	<gazebo reference="base_link">
+		<material>Gazebo/DarkGrey</material>
+	</gazebo>
+	<gazebo reference="link_b1">
+		<material>Gazebo/DarkGrey</material>
+	</gazebo>
+	<gazebo reference="link_b2">
+		<material>Gazebo/DarkGrey</material>
+	</gazebo>
+	<gazebo reference="link_b3">
+		<material>Gazebo/DarkGrey</material>
+	</gazebo>
 </robot>

File: tr2_description/urdf/base/base.urdf.xacro (robot description, xacro)
@@ -7,5 +7,5 @@
 		<joint name="${name}" type="continuous">
 			<parent link="base_link"/>
-			<child link="${name}_link"/>
+			<child link="link_${name}"/>
 		  <axis xyz="0 1 0"/>
 			<limit effort="1.0" lower="-1.0" upper="1.0" velocity="12.0"/>
@@ -13,5 +13,5 @@
     	<dynamics damping="0" friction="0"/>
 		</joint>
-		<link name="${name}_link">
+		<link name="link_${name}">
 			<collision>
 				<geometry>

File: tr2_description/urdf/head/head.gazebo.xacro (robot description, xacro)
@@ -44,3 +44,9 @@
 		</sensor>
 	</gazebo>
+	<gazebo reference="neck_link">
+		<material>Gazebo/DarkGrey</material>
+	</gazebo>
+	<gazebo reference="head_link">
+		<material>Gazebo/DarkGrey</material>
+	</gazebo>
 </robot>

File: tr2_description/urdf/head/head.urdf.xacro (robot description, xacro)
@@ -60,5 +60,5 @@
 		<parent link="head_link"/>
 		<child link="camera_link"/>
-		<origin rpy="0 0 1.5708" xyz="0 0.115 0.035"/>
+		<origin rpy="0 0 1.5708" xyz="0.025 0.150 0.0"/>
 		<axis xyz="1 0 0" />
 	</joint>
