Commit message: integration with point cloud camera

File: tr2_description/urdf/head/head.gazebo.xacro (robot description, xacro)
@@ -1,11 +1,11 @@
 <?xml version="1.0"?>
 <robot xmlns:xacro="http://www.ros.org/wiki/xacro">
-	<gazebo reference="camera_link">
+	<gazebo reference="camera_link_optical">
 		<sensor type="depth" name="orbbec_astra">
 			<always_on>1</always_on>
 			<visualize>true</visualize>
 			<camera>
-				<pose>0 0 0 0 0 0</pose>
-				<horizontal_fov>1.5807</horizontal_fov>
+				<pose>0 0 0 3.1415 -1.5708 -1.5708</pose>
+				<horizontal_fov>1.0</horizontal_fov>
 				<image>
 					<width>640</width>
@@ -16,6 +16,6 @@
 				</depth_camera>
 				<clip>
-					<near>0.1</near>
-					<far>100</far>
+					<near>0.6</near>
+					<far>8.0</far>
 				</clip>
 			</camera>
@@ -24,5 +24,5 @@
 				<updateRate>10.0</updateRate>
 				<cameraName>camera</cameraName>
-				<frameName>camera_link</frameName>
+				<frameName>camera_link_optical</frameName>
 				<imageTopicName>rgb/image_raw</imageTopicName>
 				<depthImageTopicName>depth/image_raw</depthImageTopicName>

File: tr2_description/urdf/head/head.transmission.xacro (robot description, xacro)
@@ -4,5 +4,5 @@
     <type>transmission_interface/SimpleTransmission</type>
     <actuator name="h0_actuator">
-      <mechanicalReduction>378</mechanicalReduction>
+      <mechanicalReduction>2000</mechanicalReduction>
       <hardwareInterface>EffortJointInterface</hardwareInterface>
     </actuator>
@@ -14,5 +14,5 @@
     <type>transmission_interface/SimpleTransmission</type>
     <actuator name="h1_actuator">
-      <mechanicalReduction>378</mechanicalReduction>
+      <mechanicalReduction>2000</mechanicalReduction>
       <hardwareInterface>EffortJointInterface</hardwareInterface>
     </actuator>

File: tr2_description/urdf/head/head.urdf.xacro (robot description, xacro)
@@ -57,9 +57,15 @@
     </inertial>
   </link>
+  <link name="camera_link_optical">
+  </link>
+  <joint name="camera_optical_joint" type="fixed">
+    <origin xyz="0 0 0" rpy="-1.5708 0 0"/>
+    <parent link="camera_link"/>
+    <child link="camera_link_optical"/>
+  </joint>
 	<joint name="camera_joint" type="fixed">
 		<parent link="head_link"/>
 		<child link="camera_link"/>
-		<origin rpy="0 0 1.5708" xyz="0.025 0.150 0.0"/>
-		<axis xyz="1 0 0" />
+		<origin rpy="0 0 0" xyz="0.025 0.150 0.0"/>
 	</joint>
 	<joint name="h0" type="revolute">
@@ -68,5 +74,5 @@
 		<origin xyz="0 -0.1227 0.9071"/>
     <axis xyz="0 0 1"/>
-		<limit effort="1.0" lower="-6.29" upper="6.29" velocity="1.4661"/>
+		<limit effort="100.0" lower="-15" upper="15" velocity="0.20"/>
     <dynamics damping="0.1" friction="0.1"/>
 	</joint>
@@ -76,5 +82,5 @@
 		<origin xyz="-0.0688 0.1745 0.1614" rpy="-0.3490 0 0"/>
     <axis xyz="1 0 0"/>
-		<limit effort="1.0" lower="-6.29" upper="6.29" velocity="1.4661"/>
+		<limit effort="100.0" lower="-15" upper="15" velocity="0.20"/>
     <dynamics damping="0.1" friction="0.1"/>
 	</joint>
