Commit message: object avoidance buildout

File: tr2_description/urdf/base/base.transmission.xacro (robot description, xacro)
@@ -4,5 +4,5 @@
     <type>transmission_interface/SimpleTransmission</type>
     <actuator name="motor19">
-      <mechanicalReduction>1</mechanicalReduction>
+      <mechanicalReduction>2000</mechanicalReduction>
       <hardwareInterface>EffortJointInterface</hardwareInterface>
     </actuator>
@@ -14,5 +14,5 @@
     <type>transmission_interface/SimpleTransmission</type>
     <actuator name="motor20">
-      <mechanicalReduction>1</mechanicalReduction>
+      <mechanicalReduction>2000</mechanicalReduction>
       <hardwareInterface>EffortJointInterface</hardwareInterface>
     </actuator>

File: tr2_description/urdf/base/base.urdf.xacro (robot description, xacro)
@@ -11,5 +11,5 @@
 			<limit effort="100.0" lower="-4.0" upper="4.0" velocity="4.0"/>
 			<xacro:insert_block name="origin" />
-    	<dynamics damping="1.0" friction="2.0"/>
+    	<dynamics damping="0.1" friction="0.1"/>
 		</joint>
 		<link name="link_${name}">
