Commit message: tr2 navigation refactoring, better simulation performance

File: tr2_description/urdf/base/base.urdf.xacro (robot description, xacro)
@@ -9,7 +9,7 @@
 			<child link="link_${name}"/>
 		  <axis xyz="0 1 0"/>
-			<limit effort="100.0" lower="-4.0" upper="4.0" velocity="4.0"/>
+			<limit effort="100.0" velocity="8.8"/>
 			<xacro:insert_block name="origin" />
-    	<dynamics damping="0.1" friction="0.1"/>
+    	<dynamics damping="0.001" friction="0.001"/>
 		</joint>
 		<link name="link_${name}">
@@ -21,7 +21,7 @@
 			</collision>
 			<inertial>
-				<mass value="12.0"/>
-				<inertia ixx="0.1" iyy="0.1" izz="0.1" ixy="0" ixz="0" iyz="0" />
-			</inertial>
+      	<mass value="0.01" />
+		    <inertia ixx="0.001" ixy="0.0" ixz="0.0" iyy="0.001" iyz="0.0" izz="0.001" />
+				</inertial>
 			<visual>
 				<geometry>
@@ -44,6 +44,6 @@
 		</collision>
 		<inertial>
-			<mass value="1.0"/>
-			<inertia ixx="0.1" iyy="0.1" izz="0.1" ixy="0" ixz="0" iyz="0" />
+      	<mass value="0.5" />
+		    <inertia ixx="0.001" ixy="0.0" ixz="0.0" iyy="0.001" iyz="0.0" izz="0.001" />
 		</inertial>
 		<visual>
@@ -66,6 +66,6 @@
 		</collision>
 		<inertial>
-			<mass value="1.0"/>
-			<inertia ixx="0.1" iyy="0.1" izz="0.1" ixy="0" ixz="0" iyz="0" />
+      	<mass value="0.01" />
+		    <inertia ixx="0.001" ixy="0.0" ixz="0.0" iyy="0.001" iyz="0.0" izz="0.001" />
 		</inertial>
 		<visual>
@@ -87,6 +87,6 @@
 		</collision>
 		<inertial>
-			<mass value="1.0"/>
-			<inertia ixx="0.1" iyy="0.1" izz="0.1" ixy="0" ixz="0" iyz="0" />
+      	<mass value="0.01" />
+		    <inertia ixx="0.001" ixy="0.0" ixz="0.0" iyy="0.001" iyz="0.0" izz="0.001" />
 		</inertial>
 		<visual>
